Commit message: feat: stable AAS generation for IGUS Rebel (v1.0 baseline)

File: URCell/tools/output/debug_ur10_fixed.urdf (robot description, URDF)
Before this commit: robot ur10_robot, 11 links, 10 joints
Links:
- link base_link_inertia: geometry collision mesh filename=C:/Users/benhe/desktop/abschlussarbeit/URCell/types/ur_desc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; visual mesh filename=C:/Users/benhe/desktop/abschlussarbeit/URCell/types/ur_desc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
- link forearm_link: geometry collision mesh filename=C:/Users/benhe/desktop/abschlussarbeit/URCell/types/ur_desc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; visual mesh filename=C:/Users/benhe/desktop/abschlussarbeit/URCell/types/ur_desc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
- link shoulder_link: geometry collision mesh filename=C:/Users/benhe/desktop/abschlussarbeit/URCell/types/ur_desc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; visual mesh filename=C:/Users/benhe/desktop/abschlussarbeit/URCell/types/ur_desc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
- link upper_arm_link: geometry collision mesh filename=C:/Users/benhe/desktop/abschlussarbeit/URCell/types/ur_desc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; visual mesh filename=C:/Users/benhe/desktop/abschlussarbeit/URCell/types/ur_desc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
- link wrist_1_link: geometry collision mesh filename=C:/Users/benhe/desktop/abschlussarbeit/URCell/types/ur_desc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; visual mesh filename=C:/Users/benhe/desktop/abschlussarbeit/URCell/types/ur_desc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
- link wrist_2_link: geometry collision mesh filename=C:/Users/benhe/desktop/abschlussarbeit/URCell/types/ur_desc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; visual mesh filename=C:/Users/benhe/desktop/abschlussarbeit/URCell/types/ur_desc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
- link wrist_3_link: geometry collision mesh filename=C:/Users/benhe/desktop/abschlussarbeit/URCell/types/ur_desc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; visual mesh filename=C:/Users/benhe/desktop/abschlussarbeit/URCell/types/ur_desc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

File: URCell/tools/output/debug_ur10e_fixed.urdf (robot description, URDF)
Before this commit: robot ur10e_robot, 11 links, 10 joints
Links:
- link base_link_inertia: geometry collision mesh filename=C:/Users/benhe/desktop/abschlussarbeit/URCell/types/ur_desc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; visual mesh filename=C:/Users/benhe/desktop/abschlussarbeit/URCell/types/ur_desc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
- link forearm_link: geometry collision mesh filename=C:/Users/benhe/desktop/abschlussarbeit/URCell/types/ur_desc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; visual mesh filename=C:/Users/benhe/desktop/abschlussarbeit/URCell/types/ur_desc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
- link shoulder_link: geometry collision mesh filename=C:/Users/benhe/desktop/abschlussarbeit/URCell/types/ur_desc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; visual mesh filename=C:/Users/benhe/desktop/abschlussarbeit/URCell/types/ur_desc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
- link upper_arm_link: geometry collision mesh filename=C:/Users/benhe/desktop/abschlussarbeit/URCell/types/ur_desc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; visual mesh filename=C:/Users/benhe/desktop/abschlussarbeit/URCell/types/ur_desc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
- link wrist_1_link: geometry collision mesh filename=C:/Users/benhe/desktop/abschlussarbeit/URCell/types/ur_desc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; visual mesh filename=C:/Users/benhe/desktop/abschlussarbeit/URCell/types/ur_desc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
- link wrist_2_link: geometry collision mesh filename=C:/Users/benhe/desktop/abschlussarbeit/URCell/types/ur_desc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; visual mesh filename=C:/Users/benhe/desktop/abschlussarbeit/URCell/types/ur_desc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
- link wrist_3_link: geometry collision mesh filename=C:/Users/benhe/desktop/abschlussarbeit/URCell/types/ur_desc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; visual mesh filename=C:/Users/benhe/desktop/abschlussarbeit/URCell/types/ur_desc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

File: URCell/tools/output/debug_ur12e_fixed.urdf (robot description, URDF)
Before this commit: robot ur12e_robot, 11 links, 10 joints
Links:
- link base_link_inertia: geometry collision mesh filename=C:/Users/benhe/desktop/abschlussarbeit/URCell/types/ur_desc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; visual mesh filename=C:/Users/benhe/desktop/abschlussarbeit/URCell/types/ur_desc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
- link forearm_link: geometry collision mesh filename=C:/Users/benhe/desktop/abschlussarbeit/URCell/types/ur_desc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; visual mesh filename=C:/Users/benhe/desktop/abschlussarbeit/URCell/types/ur_desc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
- link shoulder_link: geometry collision mesh filename=C:/Users/benhe/desktop/abschlussarbeit/URCell/types/ur_desc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; visual mesh filename=C:/Users/benhe/desktop/abschlussarbeit/URCell/types/ur_desc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
- link upper_arm_link: geometry collision mesh filename=C:/Users/benhe/desktop/abschlussarbeit/URCell/types/ur_desc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; visual mesh filename=C:/Users/benhe/desktop/abschlussarbeit/URCell/types/ur_desc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
- link wrist_1_link: geometry collision mesh filename=C:/Users/benhe/desktop/abschlussarbeit/URCell/types/ur_desc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; visual mesh filename=C:/Users/benhe/desktop/abschlussarbeit/URCell/types/ur_desc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
- link wrist_2_link: geometry collision mesh filename=C:/Users/benhe/desktop/abschlussarbeit/URCell/types/ur_desc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; visual mesh filename=C:/Users/benhe/desktop/abschlussarbeit/URCell/types/ur_desc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
- link wrist_3_link: geometry collision mesh filename=C:/Users/benhe/desktop/abschlussarbeit/URCell/types/ur_desc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; visual mesh filename=C:/Users/benhe/desktop/abschlussarbeit/URCell/types/ur_desc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

File: URCell/tools/output/debug_ur15_fixed.urdf (robot description, URDF)
Before this commit: robot ur15_robot, 11 links, 10 joints
Links:
- link base_link_inertia: geometry collision mesh filename=C:/Users/benhe/desktop/abschlussarbeit/URCell/types/ur_desc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; visual mesh filename=C:/Users/benhe/desktop/abschlussarbeit/URCell/types/ur_desc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
- link forearm_link: geometry collision mesh filename=C:/Users/benhe/desktop/abschlussarbeit/URCell/types/ur_desc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; visual mesh filename=C:/Users/benhe/desktop/abschlussarbeit/URCell/types/ur_desc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
- link shoulder_link: geometry collision mesh filename=C:/Users/benhe/desktop/abschlussarbeit/URCell/types/ur_desc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; visual mesh filename=C:/Users/benhe/desktop/abschlussarbeit/URCell/types/ur_desc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
- link upper_arm_link: geometry collision mesh filename=C:/Users/benhe/desktop/abschlussarbeit/URCell/types/ur_desc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; visual mesh filename=C:/Users/benhe/desktop/abschlussarbeit/URCell/types/ur_desc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
- link wrist_1_link: geometry collision mesh filename=C:/Users/benhe/desktop/abschlussarbeit/URCell/types/ur_desc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; visual mesh filename=C:/Users/benhe/desktop/abschlussarbeit/URCell/types/ur_desc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
- link wrist_2_link: geometry collision mesh filename=C:/Users/benhe/desktop/abschlussarbeit/URCell/types/ur_desc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; visual mesh filename=C:/Users/benhe/desktop/abschlussarbeit/URCell/types/ur_desc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
- link wrist_3_link: geometry collision mesh filename=C:/Users/benhe/desktop/abschlussarbeit/URCell/types/ur_desc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; visual mesh filename=C:/Users/benhe/desktop/abschlussarbeit/URCell/types/ur_desc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

File: URCell/tools/output/debug_ur16e_fixed.urdf (robot description, URDF)
Before this commit: robot ur16e_robot, 11 links, 10 joints
Links:
- link base_link_inertia: geometry collision mesh filename=C:/Users/benhe/desktop/abschlussarbeit/URCell/types/ur_desc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; visual mesh filename=C:/Users/benhe/desktop/abschlussarbeit/URCell/types/ur_desc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
- link forearm_link: geometry collision mesh filename=C:/Users/benhe/desktop/abschlussarbeit/URCell/types/ur_desc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; visual mesh filename=C:/Users/benhe/desktop/abschlussarbeit/URCell/types/ur_desc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
- link shoulder_link: geometry collision mesh filename=C:/Users/benhe/desktop/abschlussarbeit/URCell/types/ur_desc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; visual mesh filename=C:/Users/benhe/desktop/abschlussarbeit/URCell/types/ur_desc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
- link upper_arm_link: geometry collision mesh filename=C:/Users/benhe/desktop/abschlussarbeit/URCell/types/ur_desc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; visual mesh filename=C:/Users/benhe/desktop/abschlussarbeit/URCell/types/ur_desc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
- link wrist_1_link: geometry collision mesh filename=C:/Users/benhe/desktop/abschlussarbeit/URCell/types/ur_desc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; visual mesh filename=C:/Users/benhe/desktop/abschlussarbeit/URCell/types/ur_desc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
- link wrist_2_link: geometry collision mesh filename=C:/Users/benhe/desktop/abschlussarbeit/URCell/types/ur_desc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; visual mesh filename=C:/Users/benhe/desktop/abschlussarbeit/URCell/types/ur_desc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
- link wrist_3_link: geometry collision mesh filename=C:/Users/benhe/desktop/abschlussarbeit/URCell/types/ur_desc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; visual mesh filename=C:/Users/benhe/desktop/abschlussarbeit/URCell/types/ur_desc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

File: URCell/tools/output/debug_ur20_fixed.urdf (robot description, URDF)
Before this commit: robot ur20_robot, 11 links, 10 joints
Links:
- link base_link_inertia: geometry collision mesh filename=C:/Users/benhe/desktop/abschlussarbeit/URCell/types/ur_desc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; visual mesh filename=C:/Users/benhe/desktop/abschlussarbeit/URCell/types/ur_desc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
- link forearm_link: geometry collision mesh filename=C:/Users/benhe/desktop/abschlussarbeit/URCell/types/ur_desc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; visual mesh filename=C:/Users/benhe/desktop/abschlussarbeit/URCell/types/ur_desc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
- link shoulder_link: geometry collision mesh filename=C:/Users/benhe/desktop/abschlussarbeit/URCell/types/ur_desc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; visual mesh filename=C:/Users/benhe/desktop/abschlussarbeit/URCell/types/ur_desc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
- link upper_arm_link: geometry collision mesh filename=C:/Users/benhe/desktop/abschlussarbeit/URCell/types/ur_desc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; visual mesh filename=C:/Users/benhe/desktop/abschlussarbeit/URCell/types/ur_desc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
- link wrist_1_link: geometry collision mesh filename=C:/Users/benhe/desktop/abschlussarbeit/URCell/types/ur_desc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; visual mesh filename=C:/Users/benhe/desktop/abschlussarbeit/URCell/types/ur_desc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
- link wrist_2_link: geometry collision mesh filename=C:/Users/benhe/desktop/abschlussarbeit/URCell/types/ur_desc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; visual mesh filename=C:/Users/benhe/desktop/abschlussarbeit/URCell/types/ur_desc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
- link wrist_3_link: geometry collision mesh filename=C:/Users/benhe/desktop/abschlussarbeit/URCell/types/ur_desc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; visual mesh filename=C:/Users/benhe/desktop/abschlussarbeit/URCell/types/ur_desc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

File: URCell/tools/output/debug_ur30_fixed.urdf (robot description, URDF)
Before this commit: robot ur30_robot, 11 links, 10 joints
Links:
- link base_link_inertia: geometry collision mesh filename=C:/Users/benhe/desktop/abschlussarbeit/URCell/types/ur_desc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; visual mesh filename=C:/Users/benhe/desktop/abschlussarbeit/URCell/types/ur_desc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
- link forearm_link: geometry collision mesh filename=C:/Users/benhe/desktop/abschlussarbeit/URCell/types/ur_desc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; visual mesh filename=C:/Users/benhe/desktop/abschlussarbeit/URCell/types/ur_desc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
- link shoulder_link: geometry collision mesh filename=C:/Users/benhe/desktop/abschlussarbeit/URCell/types/ur_desc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; visual mesh filename=C:/Users/benhe/desktop/abschlussarbeit/URCell/types/ur_desc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
- link upper_arm_link: geometry collision mesh filename=C:/Users/benhe/desktop/abschlussarbeit/URCell/types/ur_desc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; visual mesh filename=C:/Users/benhe/desktop/abschlussarbeit/URCell/types/ur_desc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
- link wrist_1_link: geometry collision mesh filename=C:/Users/benhe/desktop/abschlussarbeit/URCell/types/ur_desc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; visual mesh filename=C:/Users/benhe/desktop/abschlussarbeit/URCell/types/ur_desc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
- link wrist_2_link: geometry collision mesh filename=C:/Users/benhe/desktop/abschlussarbeit/URCell/types/ur_desc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; visual mesh filename=C:/Users/benhe/desktop/abschlussarbeit/URCell/types/ur_desc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
- link wrist_3_link: geometry collision mesh filename=C:/Users/benhe/desktop/abschlussarbeit/URCell/types/ur_desc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; visual mesh filename=C:/Users/benhe/desktop/abschlussarbeit/URCell/types/ur_desc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

File: URCell/tools/output/debug_ur3_fixed.urdf (robot description, URDF)
Before this commit: robot ur3_robot, 11 links, 10 joints
Links:
- link base_link_inertia: geometry collision mesh filename=C:/Users/benhe/desktop/abschlussarbeit/URCell/types/ur_desc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; visual mesh filename=C:/Users/benhe/desktop/abschlussarbeit/URCell/types/ur_desc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
- link forearm_link: geometry collision mesh filename=C:/Users/benhe/desktop/abschlussarbeit/URCell/types/ur_desc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; visual mesh filename=C:/Users/benhe/desktop/abschlussarbeit/URCell/types/ur_desc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
- link shoulder_link: geometry collision mesh filename=C:/Users/benhe/desktop/abschlussarbeit/URCell/types/ur_desc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; visual mesh filename=C:/Users/benhe/desktop/abschlussarbeit/URCell/types/ur_desc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
- link upper_arm_link: geometry collision mesh filename=C:/Users/benhe/desktop/abschlussarbeit/URCell/types/ur_desc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; visual mesh filename=C:/Users/benhe/desktop/abschlussarbeit/URCell/types/ur_desc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
- link wrist_1_link: geometry collision mesh filename=C:/Users/benhe/desktop/abschlussarbeit/URCell/types/ur_desc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; visual mesh filename=C:/Users/benhe/desktop/abschlussarbeit/URCell/types/ur_desc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
- link wrist_2_link: geometry collision mesh filename=C:/Users/benhe/desktop/abschlussarbeit/URCell/types/ur_desc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; visual mesh filename=C:/Users/benhe/desktop/abschlussarbeit/URCell/types/ur_desc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
- link wrist_3_link: geometry collision mesh filename=C:/Users/benhe/desktop/abschlussarbeit/URCell/types/ur_desc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; visual mesh filename=C:/Users/benhe/desktop/abschlussarbeit/URCell/types/ur_desc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

File: URCell/tools/output/debug_ur3e_fixed.urdf (robot description, URDF)
Before this commit: robot ur3e_robot, 11 links, 10 joints
Links:
- link base_link_inertia: geometry collision mesh filename=C:/Users/benhe/desktop/abschlussarbeit/URCell/types/ur_desc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; visual mesh filename=C:/Users/benhe/desktop/abschlussarbeit/URCell/types/ur_desc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
- link forearm_link: geometry collision mesh filename=C:/Users/benhe/desktop/abschlussarbeit/URCell/types/ur_desc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; visual mesh filename=C:/Users/benhe/desktop/abschlussarbeit/URCell/types/ur_desc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
- link shoulder_link: geometry collision mesh filename=C:/Users/benhe/desktop/abschlussarbeit/URCell/types/ur_desc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; visual mesh filename=C:/Users/benhe/desktop/abschlussarbeit/URCell/types/ur_desc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
- link upper_arm_link: geometry collision mesh filename=C:/Users/benhe/desktop/abschlussarbeit/URCell/types/ur_desc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; visual mesh filename=C:/Users/benhe/desktop/abschlussarbeit/URCell/types/ur_desc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
- link wrist_1_link: geometry collision mesh filename=C:/Users/benhe/desktop/abschlussarbeit/URCell/types/ur_desc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; visual mesh filename=C:/Users/benhe/desktop/abschlussarbeit/URCell/types/ur_desc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
- link wrist_2_link: geometry collision mesh filename=C:/Users/benhe/desktop/abschlussarbeit/URCell/types/ur_desc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; visual mesh filename=C:/Users/benhe/desktop/abschlussarbeit/URCell/types/ur_desc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
- link wrist_3_link: geometry collision mesh filename=C:/Users/benhe/desktop/abschlussarbeit/URCell/types/ur_desc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; visual mesh filename=C:/Users/benhe/desktop/abschlussarbeit/URCell/types/ur_desc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

File: URCell/tools/output/debug_ur5_fixed.urdf (robot description, URDF)
Before this commit: robot ur5_robot, 11 links, 10 joints
Links:
- link base_link_inertia: geometry collision mesh filename=C:/Users/benhe/desktop/abschlussarbeit/URCell/types/ur_desc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; visual mesh filename=C:/Users/benhe/desktop/abschlussarbeit/URCell/types/ur_desc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
- link forearm_link: geometry collision mesh filename=C:/Users/benhe/desktop/abschlussarbeit/URCell/types/ur_desc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; visual mesh filename=C:/Users/benhe/desktop/abschlussarbeit/URCell/types/ur_desc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
- link shoulder_link: geometry collision mesh filename=C:/Users/benhe/desktop/abschlussarbeit/URCell/types/ur_desc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; visual mesh filename=C:/Users/benhe/desktop/abschlussarbeit/URCell/types/ur_desc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
- link upper_arm_link: geometry collision mesh filename=C:/Users/benhe/desktop/abschlussarbeit/URCell/types/ur_desc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; visual mesh filename=C:/Users/benhe/desktop/abschlussarbeit/URCell/types/ur_desc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
- link wrist_1_link: geometry collision mesh filename=C:/Users/benhe/desktop/abschlussarbeit/URCell/types/ur_desc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; visual mesh filename=C:/Users/benhe/desktop/abschlussarbeit/URCell/types/ur_desc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
- link wrist_2_link: geometry collision mesh filename=C:/Users/benhe/desktop/abschlussarbeit/URCell/types/ur_desc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; visual mesh filename=C:/Users/benhe/desktop/abschlussarbeit/URCell/types/ur_desc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
- link wrist_3_link: geometry collision mesh filename=C:/Users/benhe/desktop/abschlussarbeit/URCell/types/ur_desc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; visual mesh filename=C:/Users/benhe/desktop/abschlussarbeit/URCell/types/ur_desc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

File: URCell/tools/output/debug_ur5e_fixed.urdf (robot description, URDF)
Before this commit: robot ur5e_robot, 11 links, 10 joints
Links:
- link base_link_inertia: geometry collision mesh filename=C:/Users/benhe/desktop/abschlussarbeit/URCell/types/ur_desc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; visual mesh filename=C:/Users/benhe/desktop/abschlussarbeit/URCell/types/ur_desc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
- link forearm_link: geometry collision mesh filename=C:/Users/benhe/desktop/abschlussarbeit/URCell/types/ur_desc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; visual mesh filename=C:/Users/benhe/desktop/abschlussarbeit/URCell/types/ur_desc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
- link shoulder_link: geometry collision mesh filename=C:/Users/benhe/desktop/abschlussarbeit/URCell/types/ur_desc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; visual mesh filename=C:/Users/benhe/desktop/abschlussarbeit/URCell/types/ur_desc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
- link upper_arm_link: geometry collision mesh filename=C:/Users/benhe/desktop/abschlussarbeit/URCell/types/ur_desc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; visual mesh filename=C:/Users/benhe/desktop/abschlussarbeit/URCell/types/ur_desc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
- link wrist_1_link: geometry collision mesh filename=C:/Users/benhe/desktop/abschlussarbeit/URCell/types/ur_desc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; visual mesh filename=C:/Users/benhe/desktop/abschlussarbeit/URCell/types/ur_desc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
- link wrist_2_link: geometry collision mesh filename=C:/Users/benhe/desktop/abschlussarbeit/URCell/types/ur_desc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; visual mesh filename=C:/Users/benhe/desktop/abschlussarbeit/URCell/types/ur_desc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
- link wrist_3_link: geometry collision mesh filename=C:/Users/benhe/desktop/abschlussarbeit/URCell/types/ur_desc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; visual mesh filename=C:/Users/benhe/desktop/abschlussarbeit/URCell/types/ur_desc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

File: URCell/tools/output/debug_ur7e_fixed.urdf (robot description, URDF)
Before this commit: robot ur7e_robot, 11 links, 10 joints
Links:
- link base_link_inertia: geometry collision mesh filename=C:/Users/benhe/desktop/abschlussarbeit/URCell/types/ur_desc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; visual mesh filename=C:/Users/benhe/desktop/abschlussarbeit/URCell/types/ur_desc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
- link forearm_link: geometry collision mesh filename=C:/Users/benhe/desktop/abschlussarbeit/URCell/types/ur_desc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; visual mesh filename=C:/Users/benhe/desktop/abschlussarbeit/URCell/types/ur_desc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
- link shoulder_link: geometry collision mesh filename=C:/Users/benhe/desktop/abschlussarbeit/URCell/types/ur_desc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; visual mesh filename=C:/Users/benhe/desktop/abschlussarbeit/URCell/types/ur_desc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
- link upper_arm_link: geometry collision mesh filename=C:/Users/benhe/desktop/abschlussarbeit/URCell/types/ur_desc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; visual mesh filename=C:/Users/benhe/desktop/abschlussarbeit/URCell/types/ur_desc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
- link wrist_1_link: geometry collision mesh filename=C:/Users/benhe/desktop/abschlussarbeit/URCell/types/ur_desc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; visual mesh filename=C:/Users/benhe/desktop/abschlussarbeit/URCell/types/ur_desc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
- link wrist_2_link: geometry collision mesh filename=C:/Users/benhe/desktop/abschlussarbeit/URCell/types/ur_desc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; visual mesh filename=C:/Users/benhe/desktop/abschlussarbeit/URCell/types/ur_desc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
- link wrist_3_link: geometry collision mesh filename=C:/Users/benhe/desktop/abschlussarbeit/URCell/types/ur_desc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; visual mesh filename=C:/Users/benhe/desktop/abschlussarbeit/URCell/types/ur_desc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
