Commit message: 一个大致模板

File: URCell/projects/multi_ur(模板).xacro (robot description, xacro)
@@ -1,5 +1,5 @@
 <?xml version="1.0"?>
 <robot xmlns:xacro="http://www.ros.org/wiki/xacro" name="multi_ur">
-  <xacro:include filename="spawns/igus_rebel_6dof_spawn_hand.xacro"/>
+  <!-- 正确的 include 写法 -->
   <xacro:include filename="spawns/ur5_spawn_hand.xacro"/>
   <link name="world"/>
@@ -15,4 +15,4 @@
     <origin xyz="0 1 0" rpy="0 0 0"/>
   </joint>
-  <xacro:igus_rebel_6dof_spawn_hand prefix="robot2_" xyz="0 1 0" rpy="0 0 0"/>
+  <xacro:ur5_spawn_hand prefix="robot2_" xyz="0 1 0" rpy="0 0 0"/>
 </robot>
