Commit message: 一个大致模板

File: URCell/projects/spawns/ur5_spawn.xacro (robot description, xacro)
@@ -1,580 +1,187 @@
-<?xml version='1.0' encoding='utf-8'?>
-<robot name="UR5" xmlns:xacro="http://wiki.ros.org/xacro">
-  <!--Auto-generated pure data-driven macro (with links + transmissions)-->
-  <!--Robot: UR5-->
-  <!--Generated at: 2025-11-11 17:40:54-->
-  <xacro:macro name="ur5_spawn">
-    <link name="base_link" />
-    <link name="base_link_inertia" />
-    <link name="flange" />
-    <link name="forearm_link" />
-    <link name="shoulder_link" />
-    <link name="upper_arm_link" />
-    <link name="wrist_1_link" />
-    <link name="wrist_2_link" />
-    <link name="wrist_3_link" />
-    <joint name="Link_base_link" type="revolute">
-      <origin xyz="0 0 0" rpy="0 0 0" />
-    </joint><joint name="Link_shoulder_link" type="revolute">
-      <origin xyz="0 0 0" rpy="0 0 0" />
-    </joint><joint name="Link_upper_arm_link" type="revolute">
-      <origin xyz="0 0 0" rpy="0 0 0" />
-    </joint><joint name="Link_forearm_link" type="revolute">
-      <origin xyz="0 0 0" rpy="0 0 0" />
-    </joint><joint name="Link_wrist_1_link" type="revolute">
-      <origin xyz="0 0 0" rpy="0 0 0" />
-    </joint><joint name="Link_wrist_2_link" type="revolute">
-      <origin xyz="0 0 0" rpy="0 0 0" />
-    </joint><joint name="Link_wrist_3_link" type="revolute">
-      <origin xyz="0 0 0" rpy="0 0 0" />
-    </joint><joint name="Link_base" type="revolute">
-      <origin xyz="0 0 0" rpy="0 0 0" />
-    </joint><joint name="Link_flange" type="revolute">
-      <origin xyz="0 0 0" rpy="0 0 0" />
-    </joint><joint name="Link_tool0" type="revolute">
-      <origin xyz="0 0 0" rpy="0 0 0" />
-    </joint><joint name="Joint_base_link-base_link_inertia" type="revolute">
-      <parent link="base_link" />
-      <origin xyz="0 0 0" rpy="0 0 3.141592653589793" />
-    </joint><joint name="Joint_shoulder_pan_joint" type="revolute">
-      <parent link="base_link_inertia" />
-      <origin xyz="0 0 0.089159" rpy="0 0 0" />
-    </joint><joint name="Joint_shoulder_lift_joint" type="revolute">
-      <parent link="shoulder_link" />
-      <origin xyz="0 0 0" rpy="1.570796327 0 0" />
-    </joint><joint name="Joint_elbow_joint" type="revolute">
-      <parent link="upper_arm_link" />
-      <origin xyz="-0.425 0 0" rpy="0 0 0" />
-    </joint><joint name="Joint_wrist_1_joint" type="revolute">
-      <parent link="forearm_link" />
-      <origin xyz="-0.39225 0 0.10915" rpy="0 0 0" />
-    </joint><joint name="Joint_wrist_2_joint" type="revolute">
-      <parent link="wrist_1_link" />
-      <origin xyz="0 -0.09465 -1.941303950897609e-11" rpy="1.570796327 0 0" />
-    </joint><joint name="Joint_wrist_3_joint" type="revolute">
-      <parent link="wrist_2_link" />
-      <origin xyz="0 0.0823 -1.688001216681175e-11" rpy="1.570796326589793 3.141592653589793 3.141592653589793" />
-    </joint><joint name="Joint_base_link-base_fixed_joint" type="revolute">
-      <parent link="base_link" />
-      <origin xyz="0 0 0" rpy="0 0 3.141592653589793" />
-    </joint><joint name="Joint_wrist_3-flange" type="revolute">
-      <parent link="wrist_3_link" />
-      <origin xyz="0 0 0" rpy="0 -1.5707963267948966 -1.5707963267948966" />
-    </joint><joint name="Joint_flange-tool0" type="revolute">
-      <parent link="flange" />
-      <origin xyz="0 0 0" rpy="1.5707963267948966 0 1.5707963267948966" />
-    </joint><joint name="Joint_base_link-base_link_inertia_Control" type="revolute">
-      <origin xyz="0 0 0" rpy="0 0 0" />
-    </joint><joint name="Joint_shoulder_pan_joint_Control" type="revolute">
-      <origin xyz="0 0 0" rpy="0 0 0" />
-      <limit lower="-6.283185307179586" upper="6.283185307179586" effort="150.0" velocity="3.141592653589793" />
-    </joint><joint name="Joint_shoulder_lift_joint_Control" type="revolute">
-      <origin xyz="0 0 0" rpy="0 0 0" />
-      <limit lower="-6.283185307179586" upper="6.283185307179586" effort="150.0" velocity="3.141592653589793" />
-    </joint><joint name="Joint_elbow_joint_Control" type="revolute">
-      <origin xyz="0 0 0" rpy="0 0 0" />
-      <limit lower="-3.141592653589793" upper="3.141592653589793" effort="150.0" velocity="3.141592653589793" />
-    </joint><joint name="Joint_wrist_1_joint_Control" type="revolute">
-      <origin xyz="0 0 0" rpy="0 0 0" />
-      <limit lower="-6.283185307179586" upper="6.283185307179586" effort="28.0" velocity="3.141592653589793" />
-    </joint><joint name="Joint_wrist_2_joint_Control" type="revolute">
-      <origin xyz="0 0 0" rpy="0 0 0" />
-      <limit lower="-6.283185307179586" upper="6.283185307179586" effort="28.0" velocity="3.141592653589793" />
-    </joint><joint name="Joint_wrist_3_joint_Control" type="revolute">
-      <origin xyz="0 0 0" rpy="0 0 0" />
-      <limit lower="-6.283185307179586" upper="6.283185307179586" effort="28.0" velocity="3.141592653589793" />
-    </joint><joint name="Joint_base_link-base_fixed_joint_Control" type="revolute">
-      <origin xyz="0 0 0" rpy="0 0 0" />
-    </joint><joint name="Joint_wrist_3-flange_Control" type="revolute">
-      <origin xyz="0 0 0" rpy="0 0 0" />
-    </joint><joint name="Joint_flange-tool0_Control" type="revolute">
-      <origin xyz="0 0 0" rpy="0 0 0" />
-    </joint><joint name="Kinematics_kinematics" type="revolute">
-      <origin xyz="0 0 0" rpy="0 0 0" />
-    </joint><joint name="Dynamics_base_link" type="revolute" />
-    <joint name="Dynamics_base_link_inertia" type="revolute" />
-    <joint name="Dynamics_shoulder_link" type="revolute" />
-    <joint name="Dynamics_upper_arm_link" type="revolute" />
-    <joint name="Dynamics_forearm_link" type="revolute" />
-    <joint name="Dynamics_wrist_1_link" type="revolute" />
-    <joint name="Dynamics_wrist_2_link" type="revolute" />
-    <joint name="Dynamics_wrist_3_link" type="revolute" />
-    <joint name="Dynamics_base" type="revolute" />
-    <joint name="Dynamics_flange" type="revolute" />
-    <joint name="Dynamics_tool0" type="revolute" />
-    <joint name="Joint_shoulder_pan_joint_Safety" type="revolute">
-      <origin xyz="0 0 0" rpy="0 0 0" />
-      <limit lower="-6.283185307179586" upper="6.283185307179586" />
-    </joint><joint name="Joint_shoulder_lift_joint_Safety" type="revolute">
-      <origin xyz="0 0 0" rpy="0 0 0" />
-      <limit lower="-6.283185307179586" upper="6.283185307179586" />
-    </joint><joint name="Joint_elbow_joint_Safety" type="revolute">
-      <origin xyz="0 0 0" rpy="0 0 0" />
-      <limit lower="-3.141592653589793" upper="3.141592653589793" />
-    </joint><joint name="Joint_wrist_1_joint_Safety" type="revolute">
-      <origin xyz="0 0 0" rpy="0 0 0" />
-      <limit lower="-6.283185307179586" upper="6.283185307179586" />
-    </joint><joint name="Joint_wrist_2_joint_Safety" type="revolute">
-      <origin xyz="0 0 0" rpy="0 0 0" />
-      <limit lower="-6.283185307179586" upper="6.283185307179586" />
-    </joint><joint name="Joint_wrist_3_joint_Safety" type="revolute">
-      <origin xyz="0 0 0" rpy="0 0 0" />
-      <limit lower="-6.283185307179586" upper="6.283185307179586" />
-    </joint><joint name="Visual_base_link_inertia_0" type="revolute">
-      <origin xyz="0 0 0" rpy="0 0 0" />
-    </joint><joint name="Visual_shoulder_link_0" type="revolute">
-      <origin xyz="0 0 0" rpy="0 0 0" />
-    </joint><joint name="Visual_upper_arm_link_0" type="revolute">
-      <origin xyz="0 0 0" rpy="0 0 0" />
-    </joint><joint name="Visual_forearm_link_0" type="revolute">
-      <origin xyz="0 0 0" rpy="0 0 0" />
-    </joint><joint name="Visual_wrist_1_link_0" type="revolute">
-      <origin xyz="0 0 0" rpy="0 0 0" />
-    </joint><joint name="Visual_wrist_2_link_0" type="revolute">
-      <origin xyz="0 0 0" rpy="0 0 0" />
-    </joint><joint name="Visual_wrist_3_link_0" type="revolute">
-      <origin xyz="0 0 0" rpy="0 0 0" />
-    </joint>
-  </xacro:macro><!--Auto-generated transmission blocks-->
-  <transmission name="Link_base_link_trans">
-    <type>transmission_interface/SimpleTransmission</type>
-    <joint name="Link_base_link">
-      <hardwareInterface>hardware_interface/PositionJointInterface</hardwareInterface>
-    </joint><actuator name="Link_base_link_motor">
-      <hardwareInterface>hardware_interface/PositionJointInterface</hardwareInterface>
-      <mechanicalReduction>1</mechanicalReduction>
-    </actuator>
-  </transmission><transmission name="Link_shoulder_link_trans">
-    <type>transmission_interface/SimpleTransmission</type>
-    <joint name="Link_shoulder_link">
-      <hardwareInterface>hardware_interface/PositionJointInterface</hardwareInterface>
-    </joint><actuator name="Link_shoulder_link_motor">
-      <hardwareInterface>hardware_interface/PositionJointInterface</hardwareInterface>
-      <mechanicalReduction>1</mechanicalReduction>
-    </actuator>
-  </transmission><transmission name="Link_upper_arm_link_trans">
-    <type>transmission_interface/SimpleTransmission</type>
-    <joint name="Link_upper_arm_link">
-      <hardwareInterface>hardware_interface/PositionJointInterface</hardwareInterface>
-    </joint><actuator name="Link_upper_arm_link_motor">
-      <hardwareInterface>hardware_interface/PositionJointInterface</hardwareInterface>
-      <mechanicalReduction>1</mechanicalReduction>
-    </actuator>
-  </transmission><transmission name="Link_forearm_link_trans">
-    <type>transmission_interface/SimpleTransmission</type>
-    <joint name="Link_forearm_link">
-      <hardwareInterface>hardware_interface/PositionJointInterface</hardwareInterface>
-    </joint><actuator name="Link_forearm_link_motor">
-      <hardwareInterface>hardware_interface/PositionJointInterface</hardwareInterface>
-      <mechanicalReduction>1</mechanicalReduction>
-    </actuator>
-  </transmission><transmission name="Link_wrist_1_link_trans">
-    <type>transmission_interface/SimpleTransmission</type>
-    <joint name="Link_wrist_1_link">
-      <hardwareInterface>hardware_interface/PositionJointInterface</hardwareInterface>
-    </joint><actuator name="Link_wrist_1_link_motor">
-      <hardwareInterface>hardware_interface/PositionJointInterface</hardwareInterface>
-      <mechanicalReduction>1</mechanicalReduction>
-    </actuator>
-  </transmission><transmission name="Link_wrist_2_link_trans">
-    <type>transmission_interface/SimpleTransmission</type>
-    <joint name="Link_wrist_2_link">
-      <hardwareInterface>hardware_interface/PositionJointInterface</hardwareInterface>
-    </joint><actuator name="Link_wrist_2_link_motor">
-      <hardwareInterface>hardware_interface/PositionJointInterface</hardwareInterface>
-      <mechanicalReduction>1</mechanicalReduction>
-    </actuator>
-  </transmission><transmission name="Link_wrist_3_link_trans">
-    <type>transmission_interface/SimpleTransmission</type>
-    <joint name="Link_wrist_3_link">
-      <hardwareInterface>hardware_interface/PositionJointInterface</hardwareInterface>
-    </joint><actuator name="Link_wrist_3_link_motor">
-      <hardwareInterface>hardware_interface/PositionJointInterface</hardwareInterface>
-      <mechanicalReduction>1</mechanicalReduction>
-    </actuator>
-  </transmission><transmission name="Link_base_trans">
-    <type>transmission_interface/SimpleTransmission</type>
-    <joint name="Link_base">
-      <hardwareInterface>hardware_interface/PositionJointInterface</hardwareInterface>
-    </joint><actuator name="Link_base_motor">
-      <hardwareInterface>hardware_interface/PositionJointInterface</hardwareInterface>
-      <mechanicalReduction>1</mechanicalReduction>
-    </actuator>
-  </transmission><transmission name="Link_flange_trans">
-    <type>transmission_interface/SimpleTransmission</type>
-    <joint name="Link_flange">
-      <hardwareInterface>hardware_interface/PositionJointInterface</hardwareInterface>
-    </joint><actuator name="Link_flange_motor">
-      <hardwareInterface>hardware_interface/PositionJointInterface</hardwareInterface>
-      <mechanicalReduction>1</mechanicalReduction>
-    </actuator>
-  </transmission><transmission name="Link_tool0_trans">
-    <type>transmission_interface/SimpleTransmission</type>
-    <joint name="Link_tool0">
-      <hardwareInterface>hardware_interface/PositionJointInterface</hardwareInterface>
-    </joint><actuator name="Link_tool0_motor">
-      <hardwareInterface>hardware_interface/PositionJointInterface</hardwareInterface>
-      <mechanicalReduction>1</mechanicalReduction>
-    </actuator>
-  </transmission><transmission name="Joint_base_link-base_link_inertia_trans">
-    <type>transmission_interface/SimpleTransmission</type>
-    <joint name="Joint_base_link-base_link_inertia">
-      <hardwareInterface>hardware_interface/PositionJointInterface</hardwareInterface>
-    </joint><actuator name="Joint_base_link-base_link_inertia_motor">
-      <hardwareInterface>hardware_interface/PositionJointInterface</hardwareInterface>
-      <mechanicalReduction>1</mechanicalReduction>
-    </actuator>
-  </transmission><transmission name="Joint_shoulder_pan_joint_trans">
-    <type>transmission_interface/SimpleTransmission</type>
-    <joint name="Joint_shoulder_pan_joint">
-      <hardwareInterface>hardware_interface/PositionJointInterface</hardwareInterface>
-    </joint><actuator name="Joint_shoulder_pan_joint_motor">
-      <hardwareInterface>hardware_interface/PositionJointInterface</hardwareInterface>
-      <mechanicalReduction>1</mechanicalReduction>
-    </actuator>
-  </transmission><transmission name="Joint_shoulder_lift_joint_trans">
-    <type>transmission_interface/SimpleTransmission</type>
-    <joint name="Joint_shoulder_lift_joint">
-      <hardwareInterface>hardware_interface/PositionJointInterface</hardwareInterface>
-    </joint><actuator name="Joint_shoulder_lift_joint_motor">
-      <hardwareInterface>hardware_interface/PositionJointInterface</hardwareInterface>
-      <mechanicalReduction>1</mechanicalReduction>
-    </actuator>
-  </transmission><transmission name="Joint_elbow_joint_trans">
-    <type>transmission_interface/SimpleTransmission</type>
-    <joint name="Joint_elbow_joint">
-      <hardwareInterface>hardware_interface/PositionJointInterface</hardwareInterface>
-    </joint><actuator name="Joint_elbow_joint_motor">
-      <hardwareInterface>hardware_interface/PositionJointInterface</hardwareInterface>
-      <mechanicalReduction>1</mechanicalReduction>
-    </actuator>
-  </transmission><transmission name="Joint_wrist_1_joint_trans">
-    <type>transmission_interface/SimpleTransmission</type>
-    <joint name="Joint_wrist_1_joint">
-      <hardwareInterface>hardware_interface/PositionJointInterface</hardwareInterface>
-    </joint><actuator name="Joint_wrist_1_joint_motor">
-      <hardwareInterface>hardware_interface/PositionJointInterface</hardwareInterface>
-      <mechanicalReduction>1</mechanicalReduction>
-    </actuator>
-  </transmission><transmission name="Joint_wrist_2_joint_trans">
-    <type>transmission_interface/SimpleTransmission</type>
-    <joint name="Joint_wrist_2_joint">
-      <hardwareInterface>hardware_interface/PositionJointInterface</hardwareInterface>
-    </joint><actuator name="Joint_wrist_2_joint_motor">
-      <hardwareInterface>hardware_interface/PositionJointInterface</hardwareInterface>
-      <mechanicalReduction>1</mechanicalReduction>
-    </actuator>
-  </transmission><transmission name="Joint_wrist_3_joint_trans">
-    <type>transmission_interface/SimpleTransmission</type>
-    <joint name="Joint_wrist_3_joint">
-      <hardwareInterface>hardware_interface/PositionJointInterface</hardwareInterface>
-    </joint><actuator name="Joint_wrist_3_joint_motor">
-      <hardwareInterface>hardware_interface/PositionJointInterface</hardwareInterface>
-      <mechanicalReduction>1</mechanicalReduction>
-    </actuator>
-  </transmission><transmission name="Joint_base_link-base_fixed_joint_trans">
-    <type>transmission_interface/SimpleTransmission</type>
-    <joint name="Joint_base_link-base_fixed_joint">
-      <hardwareInterface>hardware_interface/PositionJointInterface</hardwareInterface>
-    </joint><actuator name="Joint_base_link-base_fixed_joint_motor">
-      <hardwareInterface>hardware_interface/PositionJointInterface</hardwareInterface>
-      <mechanicalReduction>1</mechanicalReduction>
-    </actuator>
-  </transmission><transmission name="Joint_wrist_3-flange_trans">
-    <type>transmission_interface/SimpleTransmission</type>
-    <joint name="Joint_wrist_3-flange">
-      <hardwareInterface>hardware_interface/PositionJointInterface</hardwareInterface>
-    </joint><actuator name="Joint_wrist_3-flange_motor">
-      <hardwareInterface>hardware_interface/PositionJointInterface</hardwareInterface>
-      <mechanicalReduction>1</mechanicalReduction>
-    </actuator>
-  </transmission><transmission name="Joint_flange-tool0_trans">
-    <type>transmission_interface/SimpleTransmission</type>
-    <joint name="Joint_flange-tool0">
-      <hardwareInterface>hardware_interface/PositionJointInterface</hardwareInterface>
-    </joint><actuator name="Joint_flange-tool0_motor">
-      <hardwareInterface>hardware_interface/PositionJointInterface</hardwareInterface>
-      <mechanicalReduction>1</mechanicalReduction>
-    </actuator>
-  </transmission><transmission name="Joint_base_link-base_link_inertia_Control_trans">
-    <type>transmission_interface/SimpleTransmission</type>
-    <joint name="Joint_base_link-base_link_inertia_Control">
-      <hardwareInterface>hardware_interface/PositionJointInterface</hardwareInterface>
-    </joint><actuator name="Joint_base_link-base_link_inertia_Control_motor">
-      <hardwareInterface>hardware_interface/PositionJointInterface</hardwareInterface>
-      <mechanicalReduction>1</mechanicalReduction>
-    </actuator>
-  </transmission><transmission name="Joint_shoulder_pan_joint_Control_trans">
-    <type>transmission_interface/SimpleTransmission</type>
-    <joint name="Joint_shoulder_pan_joint_Control">
-      <hardwareInterface>hardware_interface/PositionJointInterface</hardwareInterface>
-    </joint><actuator name="Joint_shoulder_pan_joint_Control_motor">
-      <hardwareInterface>hardware_interface/PositionJointInterface</hardwareInterface>
-      <mechanicalReduction>1</mechanicalReduction>
-    </actuator>
-  </transmission><transmission name="Joint_shoulder_lift_joint_Control_trans">
-    <type>transmission_interface/SimpleTransmission</type>
-    <joint name="Joint_shoulder_lift_joint_Control">
-      <hardwareInterface>hardware_interface/PositionJointInterface</hardwareInterface>
-    </joint><actuator name="Joint_shoulder_lift_joint_Control_motor">
-      <hardwareInterface>hardware_interface/PositionJointInterface</hardwareInterface>
-      <mechanicalReduction>1</mechanicalReduction>
-    </actuator>
-  </transmission><transmission name="Joint_elbow_joint_Control_trans">
-    <type>transmission_interface/SimpleTransmission</type>
-    <joint name="Joint_elbow_joint_Control">
-      <hardwareInterface>hardware_interface/PositionJointInterface</hardwareInterface>
-    </joint><actuator name="Joint_elbow_joint_Control_motor">
-      <hardwareInterface>hardware_interface/PositionJointInterface</hardwareInterface>
-      <mechanicalReduction>1</mechanicalReduction>
-    </actuator>
-  </transmission><transmission name="Joint_wrist_1_joint_Control_trans">
-    <type>transmission_interface/SimpleTransmission</type>
-    <joint name="Joint_wrist_1_joint_Control">
-      <hardwareInterface>hardware_interface/PositionJointInterface</hardwareInterface>
-    </joint><actuator name="Joint_wrist_1_joint_Control_motor">
-      <hardwareInterface>hardware_interface/PositionJointInterface</hardwareInterface>
-      <mechanicalReduction>1</mechanicalReduction>
-    </actuator>
-  </transmission><transmission name="Joint_wrist_2_joint_Control_trans">
-    <type>transmission_interface/SimpleTransmission</type>
-    <joint name="Joint_wrist_2_joint_Control">
-      <hardwareInterface>hardware_interface/PositionJointInterface</hardwareInterface>
-    </joint><actuator name="Joint_wrist_2_joint_Control_motor">
-      <hardwareInterface>hardware_interface/PositionJointInterface</hardwareInterface>
-      <mechanicalReduction>1</mechanicalReduction>
-    </actuator>
-  </transmission><transmission name="Joint_wrist_3_joint_Control_trans">
-    <type>transmission_interface/SimpleTransmission</type>
-    <joint name="Joint_wrist_3_joint_Control">
-      <hardwareInterface>hardware_interface/PositionJointInterface</hardwareInterface>
-    </joint><actuator name="Joint_wrist_3_joint_Control_motor">
-      <hardwareInterface>hardware_interface/PositionJointInterface</hardwareInterface>
-      <mechanicalReduction>1</mechanicalReduction>
-    </actuator>
-  </transmission><transmission name="Joint_base_link-base_fixed_joint_Control_trans">
-    <type>transmission_interface/SimpleTransmission</type>
-    <joint name="Joint_base_link-base_fixed_joint_Control">
-      <hardwareInterface>hardware_interface/PositionJointInterface</hardwareInterface>
-    </joint><actuator name="Joint_base_link-base_fixed_joint_Control_motor">
-      <hardwareInterface>hardware_interface/PositionJointInterface</hardwareInterface>
-      <mechanicalReduction>1</mechanicalReduction>
-    </actuator>
-  </transmission><transmission name="Joint_wrist_3-flange_Control_trans">
-    <type>transmission_interface/SimpleTransmission</type>
-    <joint name="Joint_wrist_3-flange_Control">
-      <hardwareInterface>hardware_interface/PositionJointInterface</hardwareInterface>
-    </joint><actuator name="Joint_wrist_3-flange_Control_motor">
-      <hardwareInterface>hardware_interface/PositionJointInterface</hardwareInterface>
-      <mechanicalReduction>1</mechanicalReduction>
-    </actuator>
-  </transmission><transmission name="Joint_flange-tool0_Control_trans">
-    <type>transmission_interface/SimpleTransmission</type>
-    <joint name="Joint_flange-tool0_Control">
-      <hardwareInterface>hardware_interface/PositionJointInterface</hardwareInterface>
-    </joint><actuator name="Joint_flange-tool0_Control_motor">
-      <hardwareInterface>hardware_interface/PositionJointInterface</hardwareInterface>
-      <mechanicalReduction>1</mechanicalReduction>
-    </actuator>
-  </transmission><transmission name="Kinematics_kinematics_trans">
-    <type>transmission_interface/SimpleTransmission</type>
-    <joint name="Kinematics_kinematics">
-      <hardwareInterface>hardware_interface/PositionJointInterface</hardwareInterface>
-    </joint><actuator name="Kinematics_kinematics_motor">
-      <hardwareInterface>hardware_interface/PositionJointInterface</hardwareInterface>
-      <mechanicalReduction>1</mechanicalReduction>
-    </actuator>
-  </transmission><transmission name="Dynamics_base_link_trans">
-    <type>transmission_interface/SimpleTransmission</type>
-    <joint name="Dynamics_base_link">
-      <hardwareInterface>hardware_interface/PositionJointInterface</hardwareInterface>
-    </joint><actuator name="Dynamics_base_link_motor">
-      <hardwareInterface>hardware_interface/PositionJointInterface</hardwareInterface>
-      <mechanicalReduction>1</mechanicalReduction>
-    </actuator>
-  </transmission><transmission name="Dynamics_base_link_inertia_trans">
-    <type>transmission_interface/SimpleTransmission</type>
-    <joint name="Dynamics_base_link_inertia">
-      <hardwareInterface>hardware_interface/PositionJointInterface</hardwareInterface>
-    </joint><actuator name="Dynamics_base_link_inertia_motor">
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