Commit message: 中文完整模型

File: URCell/projects/multi_ur.xacro (robot description, xacro)
@@ -1,6 +1,7 @@
 <?xml version="1.0"?>
 <robot xmlns:xacro="http://www.ros.org/wiki/xacro" name="multi_ur">
+  <xacro:include filename="spawns/ur5_spawn.xacro"/>
   <xacro:include filename="spawns/igus_rebel_6dof_spawn.xacro"/>
-  <xacro:include filename="spawns/ur5_spawn.xacro"/>
+  <xacro:include filename="spawns/ur3_spawn.xacro"/>
   <link name="world"/>
   <joint name="world_to_robot1" type="fixed">
@@ -16,3 +17,9 @@
   </joint>
   <xacro:igus_rebel_6dof_spawn prefix="robot2_" xyz="0 1 0" rpy="0 0 0"/>
+  <joint name="world_to_robot3" type="fixed">
+    <parent link="world"/>
+    <child link="robot3_base_link"/>
+    <origin xyz="0 3 0" rpy="0 0 0"/>
+  </joint>
+  <xacro:ur3_spawn prefix="robot3_" xyz="0 3 0" rpy="0 0 0"/>
 </robot>

File: URCell/projects/spawns/ur3_spawn.xacro (robot description, xacro)
@@ -1,6 +1,6 @@
 <?xml version="1.0"?>
 <robot xmlns:xacro="http://www.ros.org/wiki/xacro">
-<xacro:macro name="ur5_spawn_hand" params="prefix xyz rpy">
-  <xacro:property name="mesh_root" value="/home/unvrx/URCell/types/ur_description/meshes" />
+<xacro:macro name="ur3_spawn_hand" params="prefix xyz rpy">
+  <xacro:property name="mesh_root" value="/home/unvrx/URCell/types/" />
   <xacro:property name="joint_limits" value="${xacro.load_yaml('spawns/ur3_joint_limits.yaml')}" />
   <!-- LINKS -->
@@ -9,10 +9,10 @@
     <visual>
       <origin xyz="0 0 0" rpy="0 0 3.141592653589793"/>
-      <geometry><mesh filename="file://${mesh_root}/ur3/visual/base.dae"/></geometry>
+      <geometry><mesh filename="file://${mesh_root}ur_description/meshes/ur3/visual/base.dae"/></geometry>
       <material name="LightGrey"><color rgba="0.7 0.7 0.7 1.0"/></material>
     </visual>
     <collision>
       <origin xyz="0 0 0" rpy="0 0 3.141592653589793"/>
-      <geometry><mesh filename="file://${mesh_root}/ur3/collision/base.stl"/></geometry>
+      <geometry><mesh filename="file://${mesh_root}ur_description/meshes/ur3/collision/base.stl"/></geometry>
     </collision>
     <inertial>
@@ -30,10 +30,13 @@
     <visual>
 <origin xyz="0 0 0" rpy="0 0 3.141592653589793"/>
-      <geometry><mesh filename="file://${mesh_root}/ur3/visual/shoulder.dae"/></geometry>
+      <geometry><mesh filename="file://${mesh_root}ur_description/meshes/ur3/visual/shoulder.dae"/></geometry>
+      <material name="LightGrey"><color rgba="0.7 0.7 0.7 1.0"/></material>
+    </visual>
       <material name="LightGrey"><color rgba="0.7 0.7 0.7 1.0"/></material>
     </visual>
     <collision>
 <origin xyz="0 0 0" rpy="0 0 3.141592653589793"/>
-      <geometry><mesh filename="file://${mesh_root}/ur3/collision/shoulder.stl"/></geometry>
+      <geometry><mesh filename="file://${mesh_root}ur_description/meshes/ur3/collision/shoulder.stl"/></geometry>
+    </collision>
     </collision>
   </link>
@@ -46,10 +49,13 @@
     <visual>
 <origin xyz="0 0 0.1198" rpy="1.5707963267948966 0 -1.5707963267948966"/>
-      <geometry><mesh filename="file://${mesh_root}/ur3/visual/upperarm.dae"/></geometry>
+      <geometry><mesh filename="file://${mesh_root}ur_description/meshes/ur3/visual/upperarm.dae"/></geometry>
+      <material name="LightGrey"><color rgba="0.7 0.7 0.7 1.0"/></material>
+    </visual>
       <material name="LightGrey"><color rgba="0.7 0.7 0.7 1.0"/></material>
     </visual>
     <collision>
 <origin xyz="0 0 0.1198" rpy="1.5707963267948966 0 -1.5707963267948966"/>
-      <geometry><mesh filename="file://${mesh_root}/ur3/collision/upperarm.stl"/></geometry>
+      <geometry><mesh filename="file://${mesh_root}ur_description/meshes/ur3/collision/upperarm.stl"/></geometry>
+    </collision>
     </collision>
   </link>
@@ -62,10 +68,13 @@
     <visual>
 <origin xyz="0 0 0.0275" rpy="1.5707963267948966 0 -1.5707963267948966"/>
-      <geometry><mesh filename="file://${mesh_root}/ur3/visual/forearm.dae"/></geometry>
+      <geometry><mesh filename="file://${mesh_root}ur_description/meshes/ur3/visual/forearm.dae"/></geometry>
+      <material name="LightGrey"><color rgba="0.7 0.7 0.7 1.0"/></material>
+    </visual>
       <material name="LightGrey"><color rgba="0.7 0.7 0.7 1.0"/></material>
     </visual>
     <collision>
 <origin xyz="0 0 0.0275" rpy="1.5707963267948966 0 -1.5707963267948966"/>
-      <geometry><mesh filename="file://${mesh_root}/ur3/collision/forearm.stl"/></geometry>
+      <geometry><mesh filename="file://${mesh_root}ur_description/meshes/ur3/collision/forearm.stl"/></geometry>
+    </collision>
     </collision>
   </link>
@@ -78,10 +87,13 @@
     <visual>
 <origin xyz="0 0 -0.085" rpy="1.5707963267948966 0 0"/>
-      <geometry><mesh filename="file://${mesh_root}/ur3/visual/wrist1.dae"/></geometry>
+      <geometry><mesh filename="file://${mesh_root}ur_description/meshes/ur3/visual/wrist1.dae"/></geometry>
+      <material name="LightGrey"><color rgba="0.7 0.7 0.7 1.0"/></material>
+    </visual>
       <material name="LightGrey"><color rgba="0.7 0.7 0.7 1.0"/></material>
     </visual>
     <collision>
 <origin xyz="0 0 -0.085" rpy="1.5707963267948966 0 0"/>
-      <geometry><mesh filename="file://${mesh_root}/ur3/collision/wrist1.stl"/></geometry>
+      <geometry><mesh filename="file://${mesh_root}ur_description/meshes/ur3/collision/wrist1.stl"/></geometry>
+    </collision>
     </collision>
   </link>
@@ -94,10 +106,13 @@
     <visual>
 <origin xyz="0 0 -0.083" rpy="0 0 0"/>
-      <geometry><mesh filename="file://${mesh_root}/ur3/visual/wrist2.dae"/></geometry>
+      <geometry><mesh filename="file://${mesh_root}ur_description/meshes/ur3/visual/wrist2.dae"/></geometry>
+      <material name="LightGrey"><color rgba="0.7 0.7 0.7 1.0"/></material>
+    </visual>
       <material name="LightGrey"><color rgba="0.7 0.7 0.7 1.0"/></material>
     </visual>
     <collision>
 <origin xyz="0 0 -0.083" rpy="0 0 0"/>
-      <geometry><mesh filename="file://${mesh_root}/ur3/collision/wrist2.stl"/></geometry>
+      <geometry><mesh filename="file://${mesh_root}ur_description/meshes/ur3/collision/wrist2.stl"/></geometry>
+    </collision>
     </collision>
   </link>
@@ -110,10 +125,13 @@
     <visual>
 <origin xyz="0 -0.00255 -0.082" rpy="1.5707963267948966 0 0"/>
-      <geometry><mesh filename="file://${mesh_root}/ur3/visual/wrist3.dae"/></geometry>
+      <geometry><mesh filename="file://${mesh_root}ur_description/meshes/ur3/visual/wrist3.dae"/></geometry>
+      <material name="LightGrey"><color rgba="0.7 0.7 0.7 1.0"/></material>
+    </visual>
       <material name="LightGrey"><color rgba="0.7 0.7 0.7 1.0"/></material>
     </visual>
     <collision>
 <origin xyz="0 -0.00255 -0.082" rpy="1.5707963267948966 0 0"/>
-      <geometry><mesh filename="file://${mesh_root}/ur3/collision/wrist3.stl"/></geometry>
+      <geometry><mesh filename="file://${mesh_root}ur_description/meshes/ur3/collision/wrist3.stl"/></geometry>
+    </collision>
     </collision>
   </link>

File: URCell/projects/spawns/ur5_spawn.xacro (robot description, xacro)
@@ -2,5 +2,5 @@
 <robot xmlns:xacro="http://www.ros.org/wiki/xacro">
 <xacro:macro name="ur5_spawn_hand" params="prefix xyz rpy">
-  <xacro:property name="mesh_root" value="/home/unvrx/URCell/types/ur_description/meshes" />
+  <xacro:property name="mesh_root" value="/home/unvrx/URCell/types/" />
   <xacro:property name="joint_limits" value="${xacro.load_yaml('spawns/ur5_joint_limits.yaml')}" />
   <!-- LINKS -->
@@ -9,10 +9,10 @@
     <visual>
       <origin xyz="0 0 0" rpy="0 0 3.141592653589793"/>
-      <geometry><mesh filename="file://${mesh_root}/ur5/visual/base.dae"/></geometry>
+      <geometry><mesh filename="file://${mesh_root}ur_description/meshes/ur5/visual/base.dae"/></geometry>
       <material name="LightGrey"><color rgba="0.7 0.7 0.7 1.0"/></material>
     </visual>
     <collision>
       <origin xyz="0 0 0" rpy="0 0 3.141592653589793"/>
-      <geometry><mesh filename="file://${mesh_root}/ur5/collision/base.stl"/></geometry>
+      <geometry><mesh filename="file://${mesh_root}ur_description/meshes/ur5/collision/base.stl"/></geometry>
     </collision>
     <inertial>
@@ -30,10 +30,13 @@
     <visual>
 <origin xyz="0 0 0" rpy="0 0 3.141592653589793"/>
-      <geometry><mesh filename="file://${mesh_root}/ur5/visual/shoulder.dae"/></geometry>
+      <geometry><mesh filename="file://${mesh_root}ur_description/meshes/ur5/visual/shoulder.dae"/></geometry>
+      <material name="LightGrey"><color rgba="0.7 0.7 0.7 1.0"/></material>
+    </visual>
       <material name="LightGrey"><color rgba="0.7 0.7 0.7 1.0"/></material>
     </visual>
     <collision>
 <origin xyz="0 0 0" rpy="0 0 3.141592653589793"/>
-      <geometry><mesh filename="file://${mesh_root}/ur5/collision/shoulder.stl"/></geometry>
+      <geometry><mesh filename="file://${mesh_root}ur_description/meshes/ur5/collision/shoulder.stl"/></geometry>
+    </collision>
     </collision>
   </link>
@@ -46,10 +49,13 @@
     <visual>
 <origin xyz="0 0 0.13585" rpy="1.5707963267948966 0 -1.5707963267948966"/>
-      <geometry><mesh filename="file://${mesh_root}/ur5/visual/upperarm.dae"/></geometry>
+      <geometry><mesh filename="file://${mesh_root}ur_description/meshes/ur5/visual/upperarm.dae"/></geometry>
+      <material name="LightGrey"><color rgba="0.7 0.7 0.7 1.0"/></material>
+    </visual>
       <material name="LightGrey"><color rgba="0.7 0.7 0.7 1.0"/></material>
     </visual>
     <collision>
 <origin xyz="0 0 0.13585" rpy="1.5707963267948966 0 -1.5707963267948966"/>
-      <geometry><mesh filename="file://${mesh_root}/ur5/collision/upperarm.stl"/></geometry>
+      <geometry><mesh filename="file://${mesh_root}ur_description/meshes/ur5/collision/upperarm.stl"/></geometry>
+    </collision>
     </collision>
   </link>
@@ -62,10 +68,13 @@
     <visual>
 <origin xyz="0 0 0.0165" rpy="1.5707963267948966 0 -1.5707963267948966"/>
-      <geometry><mesh filename="file://${mesh_root}/ur5/visual/forearm.dae"/></geometry>
+      <geometry><mesh filename="file://${mesh_root}ur_description/meshes/ur5/visual/forearm.dae"/></geometry>
+      <material name="LightGrey"><color rgba="0.7 0.7 0.7 1.0"/></material>
+    </visual>
       <material name="LightGrey"><color rgba="0.7 0.7 0.7 1.0"/></material>
     </visual>
     <collision>
 <origin xyz="0 0 0.0165" rpy="1.5707963267948966 0 -1.5707963267948966"/>
-      <geometry><mesh filename="file://${mesh_root}/ur5/collision/forearm.stl"/></geometry>
+      <geometry><mesh filename="file://${mesh_root}ur_description/meshes/ur5/collision/forearm.stl"/></geometry>
+    </collision>
     </collision>
   </link>
@@ -78,10 +87,13 @@
     <visual>
 <origin xyz="0 0 -0.093" rpy="1.5707963267948966 0 0"/>
-      <geometry><mesh filename="file://${mesh_root}/ur5/visual/wrist1.dae"/></geometry>
+      <geometry><mesh filename="file://${mesh_root}ur_description/meshes/ur5/visual/wrist1.dae"/></geometry>
+      <material name="LightGrey"><color rgba="0.7 0.7 0.7 1.0"/></material>
+    </visual>
       <material name="LightGrey"><color rgba="0.7 0.7 0.7 1.0"/></material>
     </visual>
     <collision>
 <origin xyz="0 0 -0.093" rpy="1.5707963267948966 0 0"/>
-      <geometry><mesh filename="file://${mesh_root}/ur5/collision/wrist1.stl"/></geometry>
+      <geometry><mesh filename="file://${mesh_root}ur_description/meshes/ur5/collision/wrist1.stl"/></geometry>
+    </collision>
     </collision>
   </link>
@@ -94,10 +106,13 @@
     <visual>
 <origin xyz="0 0 -0.095" rpy="0 0 0"/>
-      <geometry><mesh filename="file://${mesh_root}/ur5/visual/wrist2.dae"/></geometry>
+      <geometry><mesh filename="file://${mesh_root}ur_description/meshes/ur5/visual/wrist2.dae"/></geometry>
+      <material name="LightGrey"><color rgba="0.7 0.7 0.7 1.0"/></material>
+    </visual>
       <material name="LightGrey"><color rgba="0.7 0.7 0.7 1.0"/></material>
     </visual>
     <collision>
 <origin xyz="0 0 -0.095" rpy="0 0 0"/>
-      <geometry><mesh filename="file://${mesh_root}/ur5/collision/wrist2.stl"/></geometry>
+      <geometry><mesh filename="file://${mesh_root}ur_description/meshes/ur5/collision/wrist2.stl"/></geometry>
+    </collision>
     </collision>
   </link>
@@ -110,10 +125,13 @@
     <visual>
 <origin xyz="0 0 -0.0818" rpy="1.5707963267948966 0 0"/>
-      <geometry><mesh filename="file://${mesh_root}/ur5/visual/wrist3.dae"/></geometry>
+      <geometry><mesh filename="file://${mesh_root}ur_description/meshes/ur5/visual/wrist3.dae"/></geometry>
+      <material name="LightGrey"><color rgba="0.7 0.7 0.7 1.0"/></material>
+    </visual>
       <material name="LightGrey"><color rgba="0.7 0.7 0.7 1.0"/></material>
     </visual>
     <collision>
 <origin xyz="0 0 -0.0818" rpy="1.5707963267948966 0 0"/>
-      <geometry><mesh filename="file://${mesh_root}/ur5/collision/wrist3.stl"/></geometry>
+      <geometry><mesh filename="file://${mesh_root}ur_description/meshes/ur5/collision/wrist3.stl"/></geometry>
+    </collision>
     </collision>
   </link>
