Commit message: Final version: confirmed and ready for submission

File: URCell/projects/multi_ur.xacro (robot description, xacro)
@@ -1,7 +1,7 @@
 <?xml version="1.0"?>
 <robot xmlns:xacro="http://www.ros.org/wiki/xacro" name="multi_ur">
-  <xacro:include filename="spawns/ur5_spawn.xacro"/>
   <xacro:include filename="spawns/igus_rebel_6dof_spawn.xacro"/>
   <xacro:include filename="spawns/ur3_spawn.xacro"/>
+  <xacro:include filename="spawns/ur5_spawn.xacro"/>
   <link name="world"/>
   <joint name="world_to_robot1" type="fixed">

File: URCell/projects/spawns/igus_rebel_6dof_spawn.xacro (robot description, xacro)
@@ -1,16 +1,17 @@
 <?xml version="1.0"?>
 <robot xmlns:xacro="http://www.ros.org/wiki/xacro">
-<xacro:macro name="igus_rebel_6dof" params="prefix xyz rpy">
-  <!-- 加载 UR5 vistion mesh -->
-<xacro:property name="mesh_root" value="/home/unvrx/URCell/types/igus_rebel_description_ros2" />
+<xacro:macro name="igus_rebel_6dof_spawn" params="prefix xyz rpy">
+  <!-- 加载 igus rebel mesh -->
+  <xacro:property name="mesh_root" value="/home/unvrx/URCell/types/igus_rebel_description_ros2" />
+  <!-- base_link -->
   <link name="${prefix}base_link">
     <visual>
       <geometry>
-        <mesh filename="file://${mesh_root}/meshes/igus_rebel_6dof_00/Joint0.dae"/>
-      </geometry>
-    </visual>
-    <collision>
-      <geometry>
-        <mesh filename="file://${mesh_root}/meshes/igus_rebel_6dof_00/Joint0Coll.dae"/>
+        <mesh filename="file://${mesh_root}/meshes/igus_rebel/Joint0.dae"/>
+      </geometry>
+    </visual>
+    <collision>
+      <geometry>
+        <mesh filename="file://${mesh_root}/meshes/igus_rebel_mod/Joint0.stl"/>
       </geometry>
     </collision>
@@ -20,7 +21,8 @@
     </inertial>
   </link>
+  <!-- joint1 -->
   <joint name="${prefix}joint1" type="revolute">
-    <parent link="base_link"/>
-    <child link="link_1"/>
+    <parent link="${prefix}base_link"/>
+    <child link="${prefix}link_1"/>
     <origin rpy="0.0 0.0 0.0" xyz="0.0 0 0.100"/>
     <axis xyz="0 0 -1"/>
@@ -30,22 +32,23 @@
     <visual>
       <geometry>
-        <mesh filename="file://${mesh_root}/meshes/igus_rebel_6dof_00/Joint1.dae"/>
-      </geometry>
-      <origin rpy="0 0 0" xyz="0 0 0"/>
-    </visual>
-    <collision>
-      <geometry>
-        <mesh filename="file://${mesh_root}/meshes/igus_rebel_6dof_00/Joint1Coll.dae"/>
-      </geometry>
-      <origin rpy="0 0 0" xyz="0 0 0"/>
-    </collision>
-    <inertial>
-      <mass value="0.1"/>
-      <inertia ixx="0.03" ixy="0.0" ixz="0.0" iyy="0.03" iyz="0.0" izz="0.03"/>
-    </inertial>
-  </link>
+        <mesh filename="file://${mesh_root}/meshes/igus_rebel/Joint1.dae"/>
+      </geometry>
+      <origin rpy="0 0 0" xyz="0 0 0"/>
+    </visual>
+    <collision>
+      <geometry>
+        <mesh filename="file://${mesh_root}/meshes/igus_rebel_mod/Joint1.stl"/>
+      </geometry>
+      <origin rpy="0 0 0" xyz="0 0 0"/>
+    </collision>
+    <inertial>
+      <mass value="0.1"/>
+      <inertia ixx="0.03" ixy="0.0" ixz="0.0" iyy="0.03" iyz="0.0" izz="0.03"/>
+    </inertial>
+  </link>
+  <!-- joint2 -->
   <joint name="${prefix}joint2" type="revolute">
-    <parent link="link_1"/>
-    <child link="link_2"/>
+    <parent link="${prefix}link_1"/>
+    <child link="${prefix}link_2"/>
     <origin rpy="0.0 0.5235987755982988 0.0" xyz="0.0 0 0.149"/>
     <axis xyz="0 1 0"/>
@@ -56,25 +59,25 @@
     <visual>
       <geometry>
-        <mesh filename="file://${mesh_root}/meshes/igus_rebel_6dof_00/Joint2.dae"/>
-      </geometry>
-      <origin rpy="0 0 0" xyz="0 0 0"/>
-    </visual>
-    <collision>
-      <geometry>
-        <mesh filename="file://${mesh_root}/meshes/igus_rebel_6dof_00/Joint2Coll.dae"/>
-      </geometry>
-      <origin rpy="0 0 0" xyz="0 0 0"/>
-    </collision>
-    <inertial>
-      <mass value="0.1"/>
-      <inertia ixx="0.03" ixy="0.0" ixz="0.0" iyy="0.03" iyz="0.0" izz="0.03"/>
-    </inertial>
-  </link>
+        <mesh filename="file://${mesh_root}/meshes/igus_rebel/Joint2.dae"/>
+      </geometry>
+      <origin rpy="0 0 0" xyz="0 0 0"/>
+    </visual>
+    <collision>
+      <geometry>
+        <mesh filename="file://${mesh_root}/meshes/igus_rebel_mod/Joint2.stl"/>
+      </geometry>
+      <origin rpy="0 0 0" xyz="0 0 0"/>
+    </collision>
+    <inertial>
+      <mass value="0.1"/>
+      <inertia ixx="0.03" ixy="0.0" ixz="0.0" iyy="0.03" iyz="0.0" izz="0.03"/>
+    </inertial>
+  </link>
+  <!-- joint3 -->
   <joint name="${prefix}joint3" type="revolute">
-    <parent link="link_2"/>
-    <child link="link_5"/>
+    <parent link="${prefix}link_2"/>
+    <child link="${prefix}link_5"/>
     <origin rpy="0.0 0.5235987755982988 0.0" xyz="0.0 0.0 0.2384"/>
     <axis xyz="0 1 0"/>
-    <!-- pi*2/3 are the physical limits, but to avoid any collisions we set the actual limits lower -->
     <limit effort="330.0" lower="-1.9198621771937623" upper="1.9198621771937623" velocity="0.7853981633974483"/>
   </joint>
@@ -82,22 +85,23 @@
     <visual>
       <geometry>
-        <mesh filename="file://${mesh_root}/meshes/igus_rebel_6dof_00/Joint3.dae"/>
-      </geometry>
-      <origin rpy="0 0 0" xyz="0 0 0"/>
-    </visual>
-    <collision>
-      <geometry>
-        <mesh filename="file://${mesh_root}/meshes/igus_rebel_6dof_00/Joint3Coll.dae"/>
-      </geometry>
-      <origin rpy="0 0 0" xyz="0 0 0"/>
-    </collision>
-    <inertial>
-      <mass value="0.1"/>
-      <inertia ixx="0.03" ixy="0.0" ixz="0.0" iyy="0.03" iyz="0.0" izz="0.03"/>
-    </inertial>
-  </link>
+        <mesh filename="file://${mesh_root}/meshes/igus_rebel/Joint3.dae"/>
+      </geometry>
+      <origin rpy="0 0 0" xyz="0 0 0"/>
+    </visual>
+    <collision>
+      <geometry>
+        <mesh filename="file://${mesh_root}/meshes/igus_rebel_mod/Joint3.stl"/>
+      </geometry>
+      <origin rpy="0 0 0" xyz="0 0 0"/>
+    </collision>
+    <inertial>
+      <mass value="0.1"/>
+      <inertia ixx="0.03" ixy="0.0" ixz="0.0" iyy="0.03" iyz="0.0" izz="0.03"/>
+    </inertial>
+  </link>
+  <!-- joint4 -->
   <joint name="${prefix}joint4" type="revolute">
-    <parent link="link_5"/>
-    <child link="link_6"/>
+    <parent link="${prefix}link_5"/>
+    <child link="${prefix}link_6"/>
     <!-- TODO The 0.03m offset are most likely caused by the mesh file (Issue 15)-->
     <origin rpy="0.0 0.0 0.0" xyz="0.0 0 0.119"/>
@@ -108,22 +112,23 @@
     <visual>
       <geometry>
-        <mesh filename="file://${mesh_root}/meshes/igus_rebel_6dof_00/Joint4.dae"/>
-      </geometry>
-      <origin rpy="0 0 0" xyz="0 0 0"/>
-    </visual>
-    <collision>
-      <geometry>
-        <mesh filename="file://${mesh_root}/meshes/igus_rebel_6dof_00/Joint4Coll.dae"/>
-      </geometry>
-      <origin rpy="0 0 0" xyz="0 0 0"/>
-    </collision>
-    <inertial>
-      <mass value="0.1"/>
-      <inertia ixx="0.03" ixy="0.0" ixz="0.0" iyy="0.03" iyz="0.0" izz="0.03"/>
-    </inertial>
-  </link>
+        <mesh filename="file://${mesh_root}/meshes/igus_rebel/Joint4.dae"/>
+      </geometry>
+      <origin rpy="0 0 0" xyz="0 0 0"/>
+    </visual>
+    <collision>
+      <geometry>
+        <mesh filename="file://${mesh_root}/meshes/igus_rebel_mod/Joint4.stl"/>
+      </geometry>
+      <origin rpy="0 0 0" xyz="0 0 0"/>
+    </collision>
+    <inertial>
+      <mass value="0.1"/>
+      <inertia ixx="0.03" ixy="0.0" ixz="0.0" iyy="0.03" iyz="0.0" izz="0.03"/>
+    </inertial>
+  </link>
+  <!-- joint5 -->
   <joint name="${prefix}joint5" type="revolute">
-    <parent link="link_6"/>
-    <child link="link_7"/>
+    <parent link="${prefix}link_6"/>
+    <child link="${prefix}link_7"/>
     <!-- TODO The 0.03m offset are most likely caused by the mesh file (Issue 15) -->
     <origin rpy="0.0 -0.1308996938995747 0.0" xyz="0.0 0 0.17"/>
@@ -134,22 +139,23 @@
     <visual>
       <geometry>
-        <mesh filename="file://${mesh_root}/meshes/igus_rebel_6dof_00/Joint5.dae"/>
-      </geometry>
-      <origin rpy="0 0 0" xyz="0 0 0"/>
-    </visual>
-    <collision>
-      <geometry>
-        <mesh filename="file://${mesh_root}/meshes/igus_rebel_6dof_00/Joint5Coll.dae"/>
-      </geometry>
-      <origin rpy="0 0 0" xyz="0 0 0"/>
-    </collision>
-    <inertial>
-      <mass value="0.1"/>
-      <inertia ixx="0.03" ixy="0.0" ixz="0.0" iyy="0.03" iyz="0.0" izz="0.03"/>
-    </inertial>
-  </link>
+        <mesh filename="file://${mesh_root}/meshes/igus_rebel/Joint5.dae"/>
+      </geometry>
+      <origin rpy="0 0 0" xyz="0 0 0"/>
+    </visual>
+    <collision>
+      <geometry>
+        <mesh filename="file://${mesh_root}/meshes/igus_rebel_mod/Joint5.stl"/>
+      </geometry>
+      <origin rpy="0 0 0" xyz="0 0 0"/>
+    </collision>
+    <inertial>
+      <mass value="0.1"/>
+      <inertia ixx="0.03" ixy="0.0" ixz="0.0" iyy="0.03" iyz="0.0" izz="0.03"/>
+    </inertial>
+  </link>
+  <!-- joint6 -->
   <joint name="${prefix}joint6" type="revolute">
-    <parent link="link_7"/>
-    <child link="link_8"/>
+    <parent link="${prefix}link_7"/>
+    <child link="${prefix}link_8"/>
     <origin rpy="0.0 0.0 0.0" xyz="0.0 0 0.1208"/>
     <axis xyz="0 0 1"/>
@@ -159,5 +165,5 @@
     <visual>
       <geometry>
-        <mesh filename="file://${mesh_root}/meshes/igus_rebel_6dof_00/Joint6.dae"/>
+        <mesh filename="file://${mesh_root}/meshes/igus_rebel/Joint6.dae"/>
       </geometry>
       <origin rpy="0 0 0" xyz="0.0 0 0"/>
@@ -165,5 +171,5 @@
     <collision>
       <geometry>
-        <mesh filename="file://${mesh_root}/meshes/igus_rebel_6dof_00/Joint6Coll.dae"/>
+        <mesh filename="file://${mesh_root}/meshes/igus_rebel_mod/Joint6.stl"/>
       </geometry>
       <origin rpy="0 0 0" xyz="0.0 0 0"/>
@@ -174,20 +180,13 @@
     </inertial>
   </link>
+  <!-- joint7 → flange -->
   <joint name="${prefix}joint7" type="fixed">
-    <parent link="link_8"/>
-    <child link="flange"/>
+    <parent link="${prefix}link_8"/>
+    <child link="${prefix}flange"/>
     <origin rpy="0.0 -1.5707963267948966 0.0" xyz="0.0 0 0.0012"/>
     <axis xyz="0 0 0"/>
   </joint>
-  <link name="${prefix}flange">
-    </link>
-  <joint name="${prefix}flange_to_tool0" type="fixed">
-    <parent link="flange"/>
-    <child link="tool0"/>
-    <origin rpy="0.0 0.0 0.0" xyz="0.0 0.0 0.0"/>
-    <axis xyz="0 0 0"/>
-  </joint>
-  <link name="${prefix}tool0">
-    </link>
+  <link name="${prefix}flange"/>
+  <!-- ros2_control -->
   <ros2_control name="igus_rebel_6dof" type="system">
     <hardware>
@@ -200,23 +199,12 @@
         <param name="max">3.12413936106985</param>
       </command_interface>
+    </joint>
   </ros2_control>
-  <!-- Add world link -->
+  <!-- world_to_base -->
   <joint name="${prefix}world_to_base" type="fixed">
     <parent link="world"/>
-    <child link="base_link"/>
+    <child link="${prefix}base_link"/>
     <origin rpy="0.0 0.0 0.0" xyz="0.0 0.0 0.0"/>
   </joint>
-  <!-- Make sure tcp exists even if no tool is attached -->
-  <joint name="${prefix}flange_to_tcp" type="fixed">
-    <parent link="flange"/>
-    <child link="tcp"/>
-    <origin rpy="0.0 0.0 0.0" xyz="0.0 0.0 0.0"/>
-    <axis xyz="0 0 0"/>
-  </joint>
-  <link name="${prefix}tcp">
-    <inertial>
-      <mass value="0.1"/>
-      <inertia ixx="0.03" ixy="0.0" ixz="0.0" iyy="0.03" iyz="0.0" izz="0.03"/>
-    </inertial>
-  </link>
+</xacro:macro>
 </robot>

File: URCell/projects/spawns/ur3_spawn.xacro (robot description, xacro)
@@ -1,7 +1,7 @@
 <?xml version="1.0"?>
 <robot xmlns:xacro="http://www.ros.org/wiki/xacro">
-<xacro:macro name="ur3_spawn_hand" params="prefix xyz rpy">
+<xacro:macro name="ur3_spawn" params="prefix xyz rpy">
   <xacro:property name="mesh_root" value="/home/unvrx/URCell/types/" />
-  <xacro:property name="joint_limits" value="${xacro.load_yaml('spawns/ur3_joint_limits.yaml')}" />
+  <xacro:property name="joint_limits" value="${xacro.load_yaml('spawns/ur3_joint_limits.yaml')}"/>
   <!-- LINKS -->
   <link name="${prefix}base_link" />
@@ -33,10 +33,7 @@
       <material name="LightGrey"><color rgba="0.7 0.7 0.7 1.0"/></material>
     </visual>
-      <material name="LightGrey"><color rgba="0.7 0.7 0.7 1.0"/></material>
-    </visual>
     <collision>
 <origin xyz="0 0 0" rpy="0 0 3.141592653589793"/>
       <geometry><mesh filename="file://${mesh_root}ur_description/meshes/ur3/collision/shoulder.stl"/></geometry>
-    </collision>
     </collision>
   </link>
@@ -52,10 +49,7 @@
       <material name="LightGrey"><color rgba="0.7 0.7 0.7 1.0"/></material>
     </visual>
-      <material name="LightGrey"><color rgba="0.7 0.7 0.7 1.0"/></material>
-    </visual>
     <collision>
 <origin xyz="0 0 0.1198" rpy="1.5707963267948966 0 -1.5707963267948966"/>
       <geometry><mesh filename="file://${mesh_root}ur_description/meshes/ur3/collision/upperarm.stl"/></geometry>
-    </collision>
     </collision>
   </link>
@@ -71,10 +65,7 @@
       <material name="LightGrey"><color rgba="0.7 0.7 0.7 1.0"/></material>
     </visual>
-      <material name="LightGrey"><color rgba="0.7 0.7 0.7 1.0"/></material>
-    </visual>
     <collision>
 <origin xyz="0 0 0.0275" rpy="1.5707963267948966 0 -1.5707963267948966"/>
       <geometry><mesh filename="file://${mesh_root}ur_description/meshes/ur3/collision/forearm.stl"/></geometry>
-    </collision>
     </collision>
   </link>
@@ -90,10 +81,7 @@
       <material name="LightGrey"><color rgba="0.7 0.7 0.7 1.0"/></material>
     </visual>
-      <material name="LightGrey"><color rgba="0.7 0.7 0.7 1.0"/></material>
-    </visual>
     <collision>
 <origin xyz="0 0 -0.085" rpy="1.5707963267948966 0 0"/>
       <geometry><mesh filename="file://${mesh_root}ur_description/meshes/ur3/collision/wrist1.stl"/></geometry>
-    </collision>
     </collision>
   </link>
@@ -109,10 +97,7 @@
       <material name="LightGrey"><color rgba="0.7 0.7 0.7 1.0"/></material>
     </visual>
-      <material name="LightGrey"><color rgba="0.7 0.7 0.7 1.0"/></material>
-    </visual>
     <collision>
 <origin xyz="0 0 -0.083" rpy="0 0 0"/>
       <geometry><mesh filename="file://${mesh_root}ur_description/meshes/ur3/collision/wrist2.stl"/></geometry>
-    </collision>
     </collision>
   </link>
@@ -128,10 +113,7 @@
       <material name="LightGrey"><color rgba="0.7 0.7 0.7 1.0"/></material>
     </visual>
-      <material name="LightGrey"><color rgba="0.7 0.7 0.7 1.0"/></material>
-    </visual>
     <collision>
 <origin xyz="0 -0.00255 -0.082" rpy="1.5707963267948966 0 0"/>
       <geometry><mesh filename="file://${mesh_root}ur_description/meshes/ur3/collision/wrist3.stl"/></geometry>
-    </collision>
     </collision>
   </link>
@@ -150,5 +132,5 @@
       lower="${joint_limits.joint_limits.shoulder_pan_joint.min_position}"
       upper="${joint_limits.joint_limits.shoulder_pan_joint.max_position}"
-      velocity="${joint_limits.joint_limits.shoulder_pan_joint.max_velocity}" />
+      velocity="${joint_limits.joint_limits.shoulder_pan_joint.max_velocity}"/>
   </joint>
   <joint name="${prefix}shoulder_lift_joint" type="revolute">
@@ -160,5 +142,5 @@
       lower="${joint_limits.joint_limits.shoulder_lift_joint.min_position}"
       upper="${joint_limits.joint_limits.shoulder_lift_joint.max_position}"
-      velocity="${joint_limits.joint_limits.shoulder_lift_joint.max_velocity}" />
+      velocity="${joint_limits.joint_limits.shoulder_lift_joint.max_velocity}"/>
   </joint>
   <joint name="${prefix}elbow_joint" type="revolute">
@@ -170,5 +152,5 @@
       lower="${joint_limits.joint_limits.elbow_joint.min_position}"
       upper="${joint_limits.joint_limits.elbow_joint.max_position}"
-      velocity="${joint_limits.joint_limits.elbow_joint.max_velocity}" />
+      velocity="${joint_limits.joint_limits.elbow_joint.max_velocity}"/>
   </joint>
   <joint name="${prefix}wrist_1_joint" type="revolute">
@@ -180,5 +162,5 @@
       lower="${joint_limits.joint_limits.wrist_1_joint.min_position}"
       upper="${joint_limits.joint_limits.wrist_1_joint.max_position}"
-      velocity="${joint_limits.joint_limits.wrist_1_joint.max_velocity}" />
+      velocity="${joint_limits.joint_limits.wrist_1_joint.max_velocity}"/>
   </joint>
   <joint name="${prefix}wrist_2_joint" type="revolute">
@@ -190,5 +172,5 @@
       lower="${joint_limits.joint_limits.wrist_2_joint.min_position}"
       upper="${joint_limits.joint_limits.wrist_2_joint.max_position}"
-      velocity="${joint_limits.joint_limits.wrist_2_joint.max_velocity}" />
+      velocity="${joint_limits.joint_limits.wrist_2_joint.max_velocity}"/>
   </joint>
   <joint name="${prefix}wrist_3_joint" type="revolute">
@@ -200,5 +182,5 @@
       lower="${joint_limits.joint_limits.wrist_3_joint.min_position}"
       upper="${joint_limits.joint_limits.wrist_3_joint.max_position}"
-      velocity="${joint_limits.joint_limits.wrist_3_joint.max_velocity}" />
+      velocity="${joint_limits.joint_limits.wrist_3_joint.max_velocity}"/>
   </joint>
 </xacro:macro>

File: URCell/projects/spawns/ur5_spawn.xacro (robot description, xacro)
@@ -1,7 +1,7 @@
 <?xml version="1.0"?>
 <robot xmlns:xacro="http://www.ros.org/wiki/xacro">
-<xacro:macro name="ur5_spawn_hand" params="prefix xyz rpy">
+<xacro:macro name="ur5_spawn" params="prefix xyz rpy">
   <xacro:property name="mesh_root" value="/home/unvrx/URCell/types/" />
-  <xacro:property name="joint_limits" value="${xacro.load_yaml('spawns/ur5_joint_limits.yaml')}" />
+  <xacro:property name="joint_limits" value="${xacro.load_yaml('spawns/ur5_joint_limits.yaml')}"/>
   <!-- LINKS -->
   <link name="${prefix}base_link" />
@@ -33,10 +33,7 @@
       <material name="LightGrey"><color rgba="0.7 0.7 0.7 1.0"/></material>
     </visual>
-      <material name="LightGrey"><color rgba="0.7 0.7 0.7 1.0"/></material>
-    </visual>
     <collision>
 <origin xyz="0 0 0" rpy="0 0 3.141592653589793"/>
       <geometry><mesh filename="file://${mesh_root}ur_description/meshes/ur5/collision/shoulder.stl"/></geometry>
-    </collision>
     </collision>
   </link>
@@ -52,10 +49,7 @@
       <material name="LightGrey"><color rgba="0.7 0.7 0.7 1.0"/></material>
     </visual>
-      <material name="LightGrey"><color rgba="0.7 0.7 0.7 1.0"/></material>
-    </visual>
     <collision>
 <origin xyz="0 0 0.13585" rpy="1.5707963267948966 0 -1.5707963267948966"/>
       <geometry><mesh filename="file://${mesh_root}ur_description/meshes/ur5/collision/upperarm.stl"/></geometry>
-    </collision>
     </collision>
   </link>
@@ -71,10 +65,7 @@
       <material name="LightGrey"><color rgba="0.7 0.7 0.7 1.0"/></material>
     </visual>
-      <material name="LightGrey"><color rgba="0.7 0.7 0.7 1.0"/></material>
-    </visual>
     <collision>
 <origin xyz="0 0 0.0165" rpy="1.5707963267948966 0 -1.5707963267948966"/>
       <geometry><mesh filename="file://${mesh_root}ur_description/meshes/ur5/collision/forearm.stl"/></geometry>
-    </collision>
     </collision>
   </link>
@@ -90,10 +81,7 @@
       <material name="LightGrey"><color rgba="0.7 0.7 0.7 1.0"/></material>
     </visual>
-      <material name="LightGrey"><color rgba="0.7 0.7 0.7 1.0"/></material>
-    </visual>
     <collision>
 <origin xyz="0 0 -0.093" rpy="1.5707963267948966 0 0"/>
       <geometry><mesh filename="file://${mesh_root}ur_description/meshes/ur5/collision/wrist1.stl"/></geometry>
-    </collision>
     </collision>
   </link>
@@ -109,10 +97,7 @@
       <material name="LightGrey"><color rgba="0.7 0.7 0.7 1.0"/></material>
     </visual>
-      <material name="LightGrey"><color rgba="0.7 0.7 0.7 1.0"/></material>
-    </visual>
     <collision>
 <origin xyz="0 0 -0.095" rpy="0 0 0"/>
       <geometry><mesh filename="file://${mesh_root}ur_description/meshes/ur5/collision/wrist2.stl"/></geometry>
-    </collision>
     </collision>
   </link>
@@ -128,10 +113,7 @@
       <material name="LightGrey"><color rgba="0.7 0.7 0.7 1.0"/></material>
     </visual>
-      <material name="LightGrey"><color rgba="0.7 0.7 0.7 1.0"/></material>
-    </visual>
     <collision>
 <origin xyz="0 0 -0.0818" rpy="1.5707963267948966 0 0"/>
       <geometry><mesh filename="file://${mesh_root}ur_description/meshes/ur5/collision/wrist3.stl"/></geometry>
-    </collision>
     </collision>
   </link>
@@ -150,5 +132,5 @@
       lower="${joint_limits.joint_limits.shoulder_pan_joint.min_position}"
       upper="${joint_limits.joint_limits.shoulder_pan_joint.max_position}"
-      velocity="${joint_limits.joint_limits.shoulder_pan_joint.max_velocity}" />
+      velocity="${joint_limits.joint_limits.shoulder_pan_joint.max_velocity}"/>
   </joint>
   <joint name="${prefix}shoulder_lift_joint" type="revolute">
@@ -160,5 +142,5 @@
       lower="${joint_limits.joint_limits.shoulder_lift_joint.min_position}"
       upper="${joint_limits.joint_limits.shoulder_lift_joint.max_position}"
-      velocity="${joint_limits.joint_limits.shoulder_lift_joint.max_velocity}" />
+      velocity="${joint_limits.joint_limits.shoulder_lift_joint.max_velocity}"/>
   </joint>
   <joint name="${prefix}elbow_joint" type="revolute">
@@ -170,5 +152,5 @@
       lower="${joint_limits.joint_limits.elbow_joint.min_position}"
       upper="${joint_limits.joint_limits.elbow_joint.max_position}"
-      velocity="${joint_limits.joint_limits.elbow_joint.max_velocity}" />
+      velocity="${joint_limits.joint_limits.elbow_joint.max_velocity}"/>
   </joint>
   <joint name="${prefix}wrist_1_joint" type="revolute">
@@ -180,5 +162,5 @@
       lower="${joint_limits.joint_limits.wrist_1_joint.min_position}"
       upper="${joint_limits.joint_limits.wrist_1_joint.max_position}"
-      velocity="${joint_limits.joint_limits.wrist_1_joint.max_velocity}" />
+      velocity="${joint_limits.joint_limits.wrist_1_joint.max_velocity}"/>
   </joint>
   <joint name="${prefix}wrist_2_joint" type="revolute">
@@ -190,5 +172,5 @@
       lower="${joint_limits.joint_limits.wrist_2_joint.min_position}"
       upper="${joint_limits.joint_limits.wrist_2_joint.max_position}"
-      velocity="${joint_limits.joint_limits.wrist_2_joint.max_velocity}" />
+      velocity="${joint_limits.joint_limits.wrist_2_joint.max_velocity}"/>
   </joint>
   <joint name="${prefix}wrist_3_joint" type="revolute">
@@ -200,5 +182,5 @@
       lower="${joint_limits.joint_limits.wrist_3_joint.min_position}"
       upper="${joint_limits.joint_limits.wrist_3_joint.max_position}"
-      velocity="${joint_limits.joint_limits.wrist_3_joint.max_velocity}" />
+      velocity="${joint_limits.joint_limits.wrist_3_joint.max_velocity}"/>
   </joint>
 </xacro:macro>
